Commit message: URDF: Resetting origin, clarifying joint rotation axis
Signed-off-by: Patrick Bertsch <47899331+pat-bert@users.noreply.github.com>

File: ressource/robot.urdf (robot description, URDF)
Before this commit: robot Mitsubishi Melfa RV-4A, 11 links, 10 joints
Joints:
- joint J2: origin xyz=1 0 0 -> (none)
- joint J3: axis (none) -> 0 0 1
- joint J4: axis (none) -> 0 0 1
- joint J5: axis (none) -> 0 0 1
- joint J6: axis (none) -> 0 0 1

Commit message: Fixed origin and link position for J1-J4
Signed-off-by: Patrick Bertsch <47899331+pat-bert@users.noreply.github.com>

File: ressource/robot.urdf (robot description, URDF)
Before this commit: robot Mitsubishi Melfa RV-4A, 11 links, 10 joints
Links:
- link base: geometry visual mesh filename=test/rv_4a_top_1_RV_4A_BASE.stl
- link link1: geometry visual mesh filename=test/rv_4a_top_1_RV_4A_SHOULDER.stl
- link link2: geometry visual mesh filename=test/rv_4a_top_1_RV_4A_NO1ARM.stl
- link link3: geometry visual mesh filename=test/rv_4a_top_1_RV_4A_ELBOW.stl
- link link4: geometry visual mesh filename=test/rv_4a_top_1_RV_4A_NO2ARM.stl
- link link4.1: geometry visual mesh filename=test/rv_4a_top_1_RV_4A_NO2ARM_LCOVER.stl
- link link4.2: geometry visual mesh filename=test/rv_4a_top_1_RV_4A_NO2ARM_RCOVER.stl
- link link5: geometry visual mesh filename=test/rv_4a_top_1_RV_4A_WRIST.stl
- link link5.1: geometry visual mesh filename=test/rv_4a_top_1_RV_4A_WRIST_RCOVER.stl
- link link5.2: geometry visual mesh filename=test/rv_4a_top_1_RV_4A_WRIST_FLANGE.stl
Joints:
- joint J1: origin (none) -> xyz=0 0 0 rpy=0 0 0
- joint J2: origin (none) -> xyz=100 0 350 rpy=-1.5708 0 0
- joint J3: origin (none) -> xyz=0 -250 0 rpy=0 0 -1.5708
- joint J4: origin (none) -> xyz=135 0 0 rpy=-1.5708 0 0

Commit message: Simplified J1-J4
Signed-off-by: Patrick Bertsch <47899331+pat-bert@users.noreply.github.com>

File: ressource/robot.urdf (robot description, URDF)
Before this commit: robot Mitsubishi Melfa RV-4A, 11 links, 10 joints
Joints:
- joint J2: axis 0 0 1 -> 0 1 0; origin xyz=100 0 350 rpy=-1.5708 0 0 -> xyz=100 0 350 rpy=0 0 0
- joint J3: axis 0 0 1 -> 0 1 0; origin xyz=0 -250 0 rpy=0 0 -1.5708 -> xyz=0 0 250 rpy=0 -1.5708 0
- joint J4: axis 0 0 1 -> 1 0 0; origin xyz=135 0 0 rpy=-1.5708 0 0 -> xyz=0 0 135 rpy=0 0 0

Commit message: Fixed origin export from SolidWorks Finalized URDF
Signed-off-by: Patrick Bertsch <47899331+pat-bert@users.noreply.github.com>

File: ressource/robot.urdf (robot description, URDF)
Before this commit: robot Mitsubishi Melfa RV-4A, 11 links, 10 joints
Links:
- removed link link5.2
- added link link6; visual mesh filename=visual/rv_4a_top_1_RV_4A_WRIST_FLANGE.stl
- link base: geometry visual mesh filename=visual/rv_4a_top_1_RV_4A_BASE.stl
- link link1: geometry visual mesh filename=visual/rv_4a_top_1_RV_4A_SHOULDER.stl
- link link2: geometry visual mesh filename=visual/rv_4a_top_1_RV_4A_NO1ARM.stl
- link link3: geometry visual mesh filename=visual/rv_4a_top_1_RV_4A_ELBOW.stl
- link link4: geometry visual mesh filename=visual/rv_4a_top_1_RV_4A_NO2ARM.stl
- link link4.1: geometry visual mesh filename=visual/rv_4a_top_1_RV_4A_NO2ARM_LCOVER.stl
- link link4.2: geometry visual mesh filename=visual/rv_4a_top_1_RV_4A_NO2ARM_RCOVER.stl
- link link5: geometry visual mesh filename=visual/rv_4a_top_1_RV_4A_WRIST.stl
- link link5.1: geometry visual mesh filename=visual/rv_4a_top_1_RV_4A_WRIST_RCOVER.stl
Joints:
- joint J5: axis 0 0 1 -> 0 1 0; origin (none) -> xyz=250 0 0 rpy=0 0 0
- joint J6: axis 0 0 1 -> 1 0 0; child tool -> link6; origin (none) -> xyz=90 0 0 rpy=0 0 0
- joint WRIST FLANGE: child link5.2 -> tool

Commit message: Added adapter plate and corrected lower limit for J3
Signed-off-by: Patrick Bertsch <47899331+pat-bert@users.noreply.github.com>

File: ressource/robot.urdf (robot description, URDF)
Before this commit: robot Mitsubishi Melfa RV-4A, 11 links, 10 joints
Links:
- added link adapter_plate; visual mesh filename=visual/adapter.stl
Joints:
- added joint INTERFACE EXTRUDER: type fixed, parent adapter_plate, child tool
- joint J3: limit lower=0 upper=2.9496 effort=0 velocity=4.7124 -> lower=0.2618 upper=2.9496 effort=0 velocity=4.7124
- joint WRIST FLANGE: child tool -> adapter_plate; parent link5 -> link6

Commit message: Removed unnecessary cover objects
Signed-off-by: Patrick Bertsch <47899331+pat-bert@users.noreply.github.com>

File: ressource/robot.urdf (robot description, URDF)
Before this commit: robot Mitsubishi Melfa RV-4A, 12 links, 11 joints
Links:
- removed link link4.1
- removed link link4.2
- removed link link5.1
- link tool: geometry visual box size=80 80 350
Joints:
- removed joint NO2ARM LEFT COVER
- removed joint NO2ARM RIGHT COVER
- removed joint WRIST REAR COVER

Commit message: Added Simscape Model and first sketch for inertial data (masses only, no accuracy required for visualization only)
Signed-off-by: Patrick Bertsch <47899331+pat-bert@users.noreply.github.com>

File: ressource/robot.urdf (robot description, URDF)
Before this commit: robot Mitsubishi Melfa RV-4A, 9 links, 8 joints
Links:
- link adapter_plate: mass None -> 0.140
- link base: mass None -> 10.842
- link link1: mass None -> 8.060
- link link2: mass None -> 5.588
- link link3: mass None -> 8.311
- link link4: mass None -> 3.204
- link link5: mass None -> 1.243
- link link6: mass None -> 0.107
- link tool: mass None -> 2

Commit message: Removed TODO from CI config URDF is now using coarse collision meshes Reduced number of triangles in meshes significantly Improved error message for passing through a singularity Changing exception in speed_profile.py Adding test gcode for passing through singularity
Signed-off-by: Patrick Bertsch <47899331+pat-bert@users.noreply.github.com>

File: ressource/robot.urdf (robot description, URDF)
Before this commit: robot Mitsubishi Melfa RV-4A, 9 links, 8 joints
Links:
- link adapter_plate: geometry visual mesh filename=collision/adapter.stl
- link base: geometry visual mesh filename=collision/rv_4a_top_1_RV_4A_BASE.stl
- link link1: geometry visual mesh filename=collision/rv_4a_top_1_RV_4A_SHOULDER.stl
- link link2: geometry visual mesh filename=collision/rv_4a_top_1_RV_4A_NO1ARM.stl
- link link3: geometry visual mesh filename=collision/rv_4a_top_1_RV_4A_ELBOW.stl
- link link4: geometry visual mesh filename=collision/rv_4a_top_1_RV_4A_NO2ARM.stl
- link link5: geometry visual mesh filename=collision/rv_4a_top_1_RV_4A_WRIST.stl
- link link6: geometry visual mesh filename=collision/rv_4a_top_1_RV_4A_WRIST_FLANGE.stl

Commit message: Adding robot cell to URDF (= static part of the env, robot is dynamic but always present, filament needs to be created dynamically) Added support for G-codes with comment in same line Added center point to circular segments Commented out error for speed profile Fixed T0 is supported Added progress bars (real parts take loong) Updated Matlab code to account for extended URDF (concave collisions cannot be checked!) -> need to update python package still
Signed-off-by: Patrick Bertsch <47899331+pat-bert@users.noreply.github.com>

File: ressource/robot.urdf (robot description, URDF)
Before this commit: robot Mitsubishi Melfa RV-4A, 9 links, 8 joints
Links:
- added link floor, mass 2; visual box size=2000 1000 50
- added link heated bed, mass 2; visual box size=400 400 50
- added link left wall, mass 2; visual box size=2000 50 1000
- added link right wall, mass 2; visual box size=2000 50 1000
Joints:
- added joint Floor connector: type fixed, parent floor, child base
- added joint Heated bed connector: type fixed, parent floor, child heated bed
- added joint Left wall connector: type fixed, parent floor, child left wall
- added joint Right wall connector: type fixed, parent floor, child right wall

Commit message: Discontinued inertial elements in URDF Optional pose flag input to coordinate conversion Sketch for singularity proximity cost
Signed-off-by: Patrick Bertsch <47899331+pat-bert@users.noreply.github.com>

File: ressource/robot.urdf (robot description, URDF)
Before this commit: robot Mitsubishi Melfa RV-4A, 13 links, 12 joints
Links:
- link adapter_plate: mass 0.140 -> None
- link base: mass 10.842 -> None
- link floor: mass 2 -> None
- link heated bed: mass 2 -> None
- link left wall: mass 2 -> None
- link link1: mass 8.060 -> None
- link link2: mass 5.588 -> None
- link link3: mass 8.311 -> None
- link link4: mass 3.204 -> None
- link link5: mass 1.243 -> None
- link link6: mass 0.107 -> None
- link right wall: mass 2 -> None
- link tool: mass 2 -> None

Commit message: Setting correct data for tool, bed origin and cell geometry
Signed-off-by: Patrick Bertsch <47899331+pat-bert@users.noreply.github.com>

File: ressource/robot.urdf (robot description, URDF)
Before this commit: robot Mitsubishi Melfa RV-4A, 13 links, 12 joints
Links:
- added link front wall; visual box size=50 800 1000
- link floor: geometry visual box size=1700 800 50
- link heated bed: geometry visual box size=400 400 38
- link left wall: geometry visual box size=1700 50 1000
- link right wall: geometry visual box size=1700 50 1000
Joints:
- added joint Front wall connector: type fixed, parent floor, child front wall

Commit message: Fixing failed print of set using comprehension in f-string Using print instead of logging for consistency Fixing sign for radial offset in DH-config Fixing collision box for extruder (only representative for lower half ^= below wrist center point) Commenting out unfinished features in prechecks
Signed-off-by: Patrick Bertsch <47899331+pat-bert@users.noreply.github.com>

File: ressource/robot.urdf (robot description, URDF)
Before this commit: robot Mitsubishi Melfa RV-4A, 14 links, 13 joints
Links:
- link tool: geometry visual box size=80 80 180
